Commit message: Eca spawns but cant be controlled yet. Behaves strangely (moves on its own). Still crashes the launch terminal. Found ROS1 code in the package

File: eca_a9_description/urdf/eca_a9_sensors.xacro (robot description, xacro)
@@ -18,17 +18,20 @@
       parent_link="${namespace}/base_link"
       inertial_reference_frame="${inertial_reference_frame}" />
+    <!-- DVL  -->
+    <!--
+    <xacro:default_dvl_macro
+      namespace="${namespace}"
+      parent_link="${namespace}/base_link"
+      inertial_reference_frame="${inertial_reference_frame}">
+      <origin xyz="-1.4 0 -0.312" rpy="0 ${0.5*pi} 0"/>
+    </xacro:default_dvl_macro>
+    -->
     <!-- DVL sensor -->
-    <xacro:dvl_plugin_macro
+    <xacro:default_dvl_macro
       namespace="${namespace}"
-      suffix=""
       parent_link="${namespace}/base_link"
-      topic="dvl"
-      scale="0.62"
-      noise_sigma="0"
-      noise_amplitude="0"
-      update_rate="7"
-      reference_frame="${inertial_reference_frame}">
+      inertial_reference_frame="${inertial_reference_frame}">
       <origin xyz="0.4785 0.0 -0.0825" rpy="0 ${0.5*pi} 0" />
-    </xacro:dvl_plugin_macro>
+    </xacro:default_dvl_macro>
     <xacro:switchable_battery_consumer_macro
       namespace="${namespace}"
@@ -120,6 +123,8 @@
       topic="${namespace}/gps/state"/>
     <!-- Mount the chemical concentration sensor -->
+    <!--
     <xacro:default_chemical_concentration_sensor namespace="${namespace}" parent_link="${namespace}/base_link">
       <origin xyz="0 0 0" rpy="0 0 0"/>
     </xacro:default_chemical_concentration_sensor>
+    -->
 </robot>
